File: schematics/PC/pc-bus.brd (EAGLE design)
At the start: 65.5 x 25.1 mm, 3 parts

Commit message: Mirror brd.
Parts:
- moved B 67.3 mm to (76.2, 40.6), turned to 270 degrees
Routing:
- net N$1: track 53.1 -> 124.2 mm
- net B0: track 124.2 -> 53.1 mm
- net N$7: track 114.1 -> 63.3 mm
- net N$2: track 63.3 -> 114.1 mm
- net N$3: track 73.4 -> 103.9 mm
- net N$6: track 103.9 -> 73.4 mm
- net N$4: track 83.6 -> 93.8 mm
- net N$5: track 93.8 -> 83.6 mm
Other:
- board size 65.5 x 25.1 mm -> 66 x 25.3 mm
