File: schematics/ALU-AXYZ/ALU.brd (EAGLE design)
At the start: 203.2 x 289.2 mm, 210 parts, among them T0 1k, T1 1k, T2 1k, T3 1k, T4 1k, T5 1k, T6 1k, T7 1k, X0 220, X1 220, X2 220, X3 220, X4 220, X5 220, X6 220, X7 220, Y0 220, Y1 220, Y2 220, Y3 220, Y4 220, Y5 220, Y6 220, Y7 220

Commit message: Added few caps to power line.
Parts:
- added C1, C2, C3, C4, C5, C6, C7, C8: (no value), rcl:E3,5-8
Connections:
- net GND: now also C1.-, C2.-, C3.-, C4.-, C5.-, C6.-, C7.-, C8.-
- net VCC: now also C1.+, C2.+, C3.+, C4.+, C5.+, C6.+, C7.+, C8.+
Routing:
- net VCC: track 1243.8 -> 1314.3 mm
- net GND: track 1918.1 -> 1985.6 mm
