File: Schematics/RAM/RAM.sch (EAGLE design)
At the start: 17 parts

Commit message: Fixed major mistakes.
Parts:
- HI, HO, LI, LO: device pinhead:PINHD-1X7 -> pinhead:PINHD-1X8
Connections:
- net A0: now also LO.8; no longer LO.7
- net A1: now also LO.7; no longer LO.6
- net A10: now also HO.6; no longer HO.4
- net A11: now also HO.5; no longer HO.3
- net A12: now also HO.4; no longer HO.2
- net A2: now also LO.6; no longer LO.5
- net A3: now also LO.5; no longer LO.4
- net A4: now also LO.4; no longer LO.3
- net A5: now also LO.3; no longer LO.2
- net A6: now also LO.2; no longer LO.1
- net A7: now also LO.1; no longer HO.7
- net A8: now also HO.8; no longer HO.6
- net A9: now also HO.7; no longer HO.5
- net B0: now also HI.8, LI.8; no longer HI.6, LI.7
- net B1: now also HI.7, LI.7; no longer HI.5, LI.6
- net B2: now also HI.6, LI.6; no longer HI.4, LI.5
- net B3: now also HI.5, LI.5; no longer HI.3, LI.4
- net B4: now also HI.4, LI.4; no longer HI.2, LI.3
- net B5: now also HI.3, LI.3; no longer HI.1, LI.2
- net B6: now also HI.2, LI.2; no longer LI.1
- net B7: now also HI.1, LI.1; no longer HI.7
Other:
- moved on the sheet: BI
