File: Schematics/RAM/reg.sch (EAGLE design)
At the start: 19 parts

Commit message: Fixed major mistakes.
Parts:
- removed BI, BO: (no value), pinhead:PINHD-1X7
- added IN, OUT: (no value), pinhead:PINHD-1X8
- added L7: (no value), led:LED5MM
- added R7: (no value), rcl:R-EU_0204/7
Connections:
- new net B7: IN.1, REG1.8D
- new net N$8: L7.A, R7.1
- new net O7: OUT.1, R7.2, REG1.8Q
- net B0: now also IN.8; no longer BI.7
- net B1: now also IN.7; no longer BI.6
- net B2: now also IN.6; no longer BI.5
- net B3: now also IN.5; no longer BI.4
- net B4: now also IN.4; no longer BI.3
- net B5: now also IN.3; no longer BI.2
- net B6: now also IN.2; no longer BI.1
- net GND: now also L7.C
- net O0: now also OUT.8; no longer BO.7
- net O1: now also OUT.7; no longer BO.6
- net O2: now also OUT.6; no longer BO.5
- net O3: now also OUT.5; no longer BO.4
- net O4: now also OUT.4; no longer BO.3
- net O5: now also OUT.3; no longer BO.2
- net O6: now also OUT.2; no longer BO.1
Other:
- moved on the sheet: CP, PS, REG/+UB, REG/-UB
