File: Schematics/B-OUT/bus.brd (EAGLE design)
At the start: 116.6 x 47 mm, 39 parts

Commit message: Added bus, fixed C1 on ALU-CTRL, CLK.zip, added 7410 to ctrl so bus out will work*.
Parts:
- removed BI, BO, BO1: (no value), pinhead:1X08
- removed C1: (no value), rcl:E2,5-6
- removed LB0, LB1, LB2, LB3, LB4, LB5, LB6, LB7, LR0, LR1, LR2, LR3, LR4, LR5, LR6, LR7: (no value), led:LED5MM
- removed OR: 74273N, 74ttl-din:DIL20
- removed OUT-CP: (no value), pinhead:1X01
- removed RB0, RB1, RB2, RB3, RB4, RB5, RB6, RB7, RR0, RR1, RR2, RR3, RR4, RR5, RR6, RR7: (no value), rcl:0204/7
- added ALU-PS, CTRL-PS, OUT-PS, PC-PS, RAM-PS, REG-PS: (no value), pinhead:1X02
- added ALU0, ALU1, CTRL, OUT, PC0, PC1, RAM0, RAM1, REG0, REG1: (no value), pinhead:1X08
- added LED1: (no value), led:LED5MM
- added R1: (no value), rcl:0204/7
- PS: device pinhead:1X02 -> con-jack:SPC4077
- moved PS 383.1 mm to (15.2, 426.7)
Connections:
- removed net CLK: OR.11, OUT-CP.1
- removed net N$10: LB3.A, RB3.1
- removed net N$11: BO.8, BO1.8, OR.19, RR7.2
- removed net N$12: LR6.A, RR6.1
- removed net N$14: BO.7, BO1.7, OR.16, RR6.2
- removed net N$15: LR5.A, RR5.1
- removed net N$16: LB2.A, RB2.1
- removed net N$17: BO.6, BO1.6, OR.15, RR5.2
- removed net N$18: LR4.A, RR4.1
- removed net N$20: BO.5, BO1.5, OR.12, RR4.2
- removed net N$21: LR3.A, RR3.1
- removed net N$22: LB1.A, RB1.1
- removed net N$23: BO.4, BO1.4, OR.9, RR3.2
- removed net N$24: LR2.A, RR2.1
- removed net N$26: BO.3, BO1.3, OR.6, RR2.2
- removed net N$27: LR1.A, RR1.1
- removed net N$28: LB0.A, RB0.1
- removed net N$29: BO.2, BO1.2, OR.5, RR1.2
- removed net N$3: LB6.A, RB6.1
- removed net N$30: LR0.A, RR0.1
- removed net N$32: BO.1, BO1.1, OR.2, RR0.2
- removed net N$5: LB5.A, RB5.1
- removed net N$7: LB4.A, RB4.1
- removed net N$9: LR7.A, RR7.1
- net B0: now also ALU0.8, ALU1.1, CTRL.1, OUT.8, PC0.1, PC1.1, RAM0.1, RAM1.1, REG0.8, REG1.8; no longer BI.8, OR.3, RB0.2
- net B1: now also ALU0.7, ALU1.2, CTRL.2, OUT.7, PC0.2, PC1.2, RAM0.2, RAM1.2, REG0.7, REG1.7; no longer BI.7, OR.4, RB1.2
- net B2: now also ALU0.6, ALU1.3, CTRL.3, OUT.6, PC0.3, PC1.3, RAM0.3, RAM1.3, REG0.6, REG1.6; no longer BI.6, OR.7, RB2.2
- net B3: now also ALU0.5, ALU1.4, CTRL.4, OUT.5, PC0.4, PC1.4, RAM0.4, RAM1.4, REG0.5, REG1.5; no longer BI.5, OR.8, RB3.2
- net B4: now also ALU0.4, ALU1.5, CTRL.5, OUT.4, PC0.5, PC1.5, RAM0.5, RAM1.5, REG0.4, REG1.4; no longer BI.4, OR.13, RB4.2
- net B5: now also ALU0.3, ALU1.6, CTRL.6, OUT.3, PC0.6, PC1.6, RAM0.6, RAM1.6, REG0.3, REG1.3; no longer BI.3, OR.14, RB5.2
- net B6: now also ALU0.2, ALU1.7, CTRL.7, OUT.2, PC0.7, PC1.7, RAM0.7, RAM1.7, REG0.2, REG1.2; no longer BI.2, OR.17, RB6.2
- net B7: now also ALU0.1, ALU1.8, CTRL.8, OUT.1, PC0.8, PC1.8, RAM0.8, RAM1.8, REG0.1, REG1.1; no longer BI.1, OR.18, RB7.2
- net GND: now also ALU-PS.1, CTRL-PS.2, LED1.K, OUT-PS.2, PC-PS.1, PS.2, RAM-PS.2, REG-PS.1; no longer C1.-, LB0.K, LB1.K, LB2.K, LB3.K, LB4.K, LB5.K, LB6.K, LB7.K, LR0.K, LR1.K, LR2.K, LR3.K, LR4.K, LR5.K, LR6.K, LR7.K, OR.10
- net N$1: now also LED1.A, R1.2; no longer LB7.A, RB7.1
- net VCC: now also ALU-PS.2, CTRL-PS.1, OUT-PS.1, PC-PS.2, PS.3, R1.1, RAM-PS.1, REG-PS.2; no longer C1.+, OR.1, OR.20, PS.2
Routing:
- net B0: track 55.4 -> 638.7 mm, vias 0 -> 9
- net B1: track 60.0 -> 640.7 mm, vias 0 -> 10
- net B2: track 68.9 -> 643.2 mm, vias 0 -> 10
- net B3: track 73.8 -> 645.8 mm, vias 0 -> 10
- net B5: track 90.1 -> 650.9 mm, vias 0 -> 10
- net B6: track 102.2 -> 654.4 mm, vias 0 -> 9
- net B4: track 96.3 -> 648.3 mm, vias 0 -> 10
- net B7: track 111.9 -> 658.3 mm, vias 0 -> 5
- net VCC: track 26.7 -> 570.8 mm, vias 0 -> 1
- net GND: track 158.9 -> 566.7 mm, vias 0 -> 6
- net N$14: track 85.7 -> 0.00 mm
- net N$32: track 84.5 -> 0.00 mm
- net N$17: track 80.8 -> 0.00 mm
- net N$11: track 78.3 -> 0.00 mm
- net N$20: track 78.0 -> 0.00 mm
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Other:
- board size 116.6 x 47 mm -> 58.4 x 434 mm
