File: Schematics/CTRL/CTRL-new.brd (EAGLE design)
At the start: 218.4 x 149.5 mm, 117 parts

Commit message: fixet version of new ctrl
Connections:
- new net NCLK: V10.10, V10.13, V10.2, V10.5, V15.10, V15.13, V15.2, V15.5, V16.2, V16.5, V6.1, V6.6, V9.12
- new net RL: IR.11, V9.11
- net CLK: now also V6.5; no longer V10.10, V10.13, V10.2, V10.5, V15.10, V15.13, V15.2, V15.5, V16.2, V16.5, V6.1, V9.1
- net GND: now also IC1.20, IC2.20, IC3.20, IC4.20
- net INC: now also V6.4
- net N$13: now also V9.1
- net RLD: now also V9.13; no longer IR.11
- net VCC: no longer IC1.20, IC2.20, IC3.20, IC4.20
Routing:
- net NCLK: track 0.00 -> 363.7 mm, vias 0 -> 5
- net INC: track 28.7 -> 207.2 mm, vias 1 -> 3
- net CLK: track 393.2 -> 216.4 mm, vias 4 -> 2
- net RL: track 0.00 -> 161.0 mm, vias 0 -> 5
- net RLD: track 210.4 -> 130.4 mm, vias 7 -> 5
- net GND: track 977.1 -> 1046.1 mm, vias 10 -> 13
- net VCC: track 906.1 -> 881.6 mm, vias 25 -> 26
- net N$13: track 52.0 -> 54.5 mm
- net C1: track 251.8 -> 252.8 mm

Commit message: fixed PLD
Parts:
- removed V7: 7400N, 74ttl-din:DIL14
- added V19: 7408N, 74ttl-din:DIL14
- V11: value 7400N -> 7408N
- moved V11 12.7 mm to (36.8, 137.2)
Connections:
- new net N$54: V13.8, V18.5
- net EF: now also V11.13; no longer V7.13
- net GF: now also V11.10; no longer V7.10
- net GND: now also V19.7; no longer V7.7
- net LF: now also V11.5; no longer V7.5
- net N$100: now also V19.8; no longer V11.8
- net N$14: now also V19.10, V19.9; no longer V11.10, V11.9
- net N$34: now also V19.12, V19.13; no longer V11.12, V11.13
- net N$35: now also V19.4; no longer V11.4
- net N$36: now also V19.1; no longer V11.1
- net N$37: now also V11.12; no longer V7.12
- net N$38: now also V11.9; no longer V7.9
- net N$39: now also V11.4; no longer V7.4
- net N$40: now also V11.1; no longer V7.1
- net N$89: now also V11.3; no longer V7.3
- net N$90: now also V11.6; no longer V7.6
- net N$91: now also V11.8; no longer V7.8
- net N$92: now also V11.11; no longer V7.11
- net N$93: now also V19.3; no longer V11.3
- net N$94: now also V19.6; no longer V11.6
- net N$99: now also V19.11; no longer V11.11
- net NG: now also V19.5; no longer V11.5
- net OF: now also V19.2; no longer V11.2
- net PLD1: now also V18.6; no longer V13.8
- net VCC: now also V19.14; no longer V7.14
- net ZF: now also V11.2; no longer V7.2
Routing:
- net PLD1: track 185.0 -> 108.4 mm, vias 5 -> 6
- net N$54: track 0.00 -> 69.2 mm, vias 0 -> 5
- net N$47: track 51.2 -> 53.3 mm
- net N$100: track 36.0 -> 36.7 mm
