File: Schematics/CTRL/CTRL.brd (EAGLE design)
At the start: 328.9 x 291.8 mm, 50 parts

Commit message: Last (probably) changes to CTRL brd.
Parts:
- removed 0X00, 0XFE, 0XFF: 74245N, 74ttl-din:DIL20
- removed ALU-CLK, PC-CLK, PC-CLR, RAM-CLK, REG-CLK: (no value), pinhead:1X01
- removed ALU-OP0, REG-OP: (no value), pinhead:1X30
- removed ALU-OP1, ALU-T, INC3, INC4: (no value), pinhead:1X05
- removed ALU-PS, PC-OP1, PC-PS, RAM-PS, REG-PS: (no value), pinhead:1X02
- removed BUS, INC1, INC2, INC7, INC8, RAM-T: (no value), pinhead:1X08
- removed C2, C3, C4, C5, C6, C7: (no value), rcl:E2,5-6
- removed DECODER: (no value), pinhead:1X11
- removed INC0: (no value), pinhead:1X07
- removed INC5, INC6: (no value), pinhead:1X06
- removed PC-OP0: (no value), pinhead:1X24
- removed PC-T: (no value), pinhead:1X10
- removed RAM-OP: (no value), pinhead:1X16
- removed REG-T: (no value), pinhead:1X03
- removed TRING: (no value), pinhead:1X15
- added ACP, ADD, AND, AOCP, AOE, AOOE, FCP, LC0, LC1, LC2, LC3, LIR0, LIR1, LIR2, LIR3, LIR4, LIR5, LIR6, NOT, OR, PCLR, PHCP, PHOE, PINC, PLCP, PLD, PLOE, POE, RHCP, RLCP, RLD, ROE, RWE, SUB, XCP, XOE, XOR, YCP, YOE: (no value), led:LED5MM
- added ALU: (no value), pinhead:2X07
- added BUSIN: (no value), pinhead:1X08
- added FLAG, RAM, REG: (no value), pinhead:2X03
- added HLT, OCP-P: (no value), pinhead:1X01
- added IC1, IC2, IC3, IC4: (no value), memory-nec:DIL28-6
- added IR: 74273N, 74ttl-din:DIL20
- added PC: (no value), pinhead:2X04
- added R1, R10, R11, R12, R13, R14, R15, R16, R17, R18, R19, R20, R21, R22, R23, R24, R25, R26, R27, R28, R29, R3, R30, R4, R5, R6, R7, R8, R9: (no value), resistor:0204/7
- added R2: (no value), rcl:0207/10
- added RC0, RC1, RC2, RC3, RIR0, RIR1, RIR2, RIR3, RIR4, RIR5, RIR6: (no value), rcl:0204/7
- added S1: (no value), switch-omron:B3F-10XX
- added V10, V15, V16, V6, V9: 7400N, 74ttl-din:DIL14
- added V11, V19: 7408N, 74ttl-din:DIL14
- added V12, V13: 7432N, 74ttl-din:DIL14
- added V14: 74193N, 74ttl-din:DIL16
- added V17, V18: 7404N, 74ttl-din:DIL14
- added V8: 74138N, 74ttl-din:DIL16
- C1: device rcl:E2,5-6 -> rcl:C050-035X075
- CLK: device pinhead:1X02 -> pinhead:1X01
- OCP: device pinhead:1X01 -> led:LED5MM
- V1: value 7400N -> 74193N; device 74ttl-din:DIL14 -> 74ttl-din:DIL16
- V2, V5: value 7410N -> 74273N; device 74ttl-din:DIL14 -> 74ttl-din:DIL20
- V3: value 7430N -> 74273N; device 74ttl-din:DIL14 -> 74ttl-din:DIL20
- V4: value 7408N -> 74273N; device 74ttl-din:DIL14 -> 74ttl-din:DIL20
- moved CLK-PS 243.1 mm to (83.8, 141.0), turned to 0 degrees
- moved V4 239.8 mm to (85.1, 57.1)
- moved V5 239.8 mm to (38.1, 57.1), turned to 0 degrees
- moved CLK 196.6 mm to (90.2, 141.0), turned to 0 degrees
- moved V3 193.4 mm to (143.5, 57.1), turned to 0 degrees
- moved V1 192.8 mm to (128.9, 127.5)
- moved V2 165.3 mm to (191.8, 57.1)
- moved PS 145.5 mm to (214.6, 133.3), turned to 270 degrees
- moved C1 143.6 mm to (154.9, 133.3), turned to 0 degrees
- moved OCP 122.3 mm to (215.3, 37.5), turned to 270 degrees
Connections:
- removed net 0X00: 0X00.19, V1.3
- removed net 0XFE: 0XFE.19, V4.6
- removed net 0XFF: 0XFF.19, V4.3
- removed net ADA: ALU-OP0.25, INC3.3
- removed net ADI: ALU-OP0.24, INC3.2, PC-OP0.12, RAM-OP.5
- removed net ADV: ALU-OP0.23, INC3.1, PC-OP0.11
- removed net ADX: ALU-OP0.27, INC3.5, REG-OP.22
- removed net ADY: ALU-OP0.26, INC3.4, REG-OP.21
- removed net ANA: ALU-OP0.9, INC7.6
- removed net ANV: ALU-OP0.8, INC7.5, PC-OP0.2
- removed net ANX: ALU-OP0.11, INC7.8, REG-OP.8
- removed net ANY: ALU-OP0.10, INC7.7, REG-OP.7
- removed net CALL: INC1.4, PC-OP0.23, RAM-OP.16, V3.1
- removed net CLA: ALU-OP0.30, INC0.4, V2.1
- removed net CLR: PC-CLR.1, TRING.1
- removed net CLX: INC0.6, REG-OP.30, V2.2
- removed net CLY: INC0.5, REG-OP.29, V2.13
- removed net CMA: ALU-OP0.28, INC1.6
- removed net CMV: INC1.5, PC-OP0.24
- removed net CMX: INC1.8, REG-OP.26
- removed net CMY: INC1.7, REG-OP.25
- removed net IRCP: DECODER.11, V1.11
- removed net JE: INC2.3, PC-OP0.14, RAM-OP.7, V3.11, V3.12
- removed net JG: INC2.4, PC-OP0.16, RAM-OP.8, V3.5
- removed net JL: INC2.5, PC-OP0.15, RAM-OP.9, V3.6
- removed net JN: INC2.6, PC-OP0.17, RAM-OP.10, V3.4
- removed net JNZ: INC2.7, PC-OP0.18, RAM-OP.11, V3.3
- removed net JZ: INC2.8, PC-OP0.19, RAM-OP.12, V3.2
- removed net L1: V1.10, V1.4, V5.8
- removed net LDA: ALU-OP0.17, INC5.4, PC-OP0.6
- removed net LDAI: ALU-OP0.16, INC5.1, PC-OP0.3, RAM-OP.1
- removed net LDX: INC5.6, PC-OP0.8, REG-OP.18
- removed net LDXI: INC5.3, PC-OP0.5, RAM-OP.3, REG-OP.16
- removed net LDY: INC5.5, PC-OP0.7, REG-OP.17
- removed net LDYI: INC5.2, PC-OP0.4, RAM-OP.2, REG-OP.15
- removed net MAX: ALU-OP0.13, INC6.2, REG-OP.10
- removed net MAY: ALU-OP0.12, INC6.1, REG-OP.9
- removed net MXA: ALU-OP0.15, INC6.5, REG-OP.13
- removed net MXY: INC6.6, REG-OP.14
- removed net MYA: ALU-OP0.14, INC6.3, REG-OP.11
- removed net MYX: INC6.4, REG-OP.12
- removed net NOA: ALU-OP1.2, INC8.2
- removed net NOP: INC0.7
- removed net NOV: ALU-OP1.1, INC8.1, PC-OP1.1
- removed net NOX: ALU-OP1.4, INC8.4, REG-OP.2
- removed net NOY: ALU-OP1.3, INC8.3, REG-OP.1
- removed net ORA: ALU-OP0.5, INC7.2
- removed net ORV: ALU-OP0.4, INC7.1, PC-OP0.1
- removed net ORX: ALU-OP0.7, INC7.4, REG-OP.6
- removed net ORY: ALU-OP0.6, INC7.3, REG-OP.5
- removed net OUA: ALU-OP0.29, INC0.1, V5.5
- removed net OUX: INC0.3, REG-OP.28, V5.3
- removed net OUY: INC0.2, REG-OP.27, V5.4
- removed net RET: INC2.2, PC-OP0.13, RAM-OP.6, V5.10, V5.11, V5.9
- removed net STA: INC1.1, PC-OP0.20, RAM-OP.13
- removed net STX: INC1.3, PC-OP0.22, RAM-OP.15, REG-OP.24
- removed net STY: INC1.2, PC-OP0.21, RAM-OP.14, REG-OP.23
- removed net SUA: ALU-OP0.20, INC4.3
- removed net SUI: ALU-OP0.19, INC4.2, PC-OP0.10, RAM-OP.4
- removed net SUV: ALU-OP0.18, INC4.1, PC-OP0.9
- removed net SUX: ALU-OP0.22, INC4.5, REG-OP.20
- removed net SUY: ALU-OP0.21, INC4.4, REG-OP.19
- removed net T0: PC-T.10, TRING.15
- removed net T1: PC-T.9, TRING.14, V1.13
- removed net T10: PC-T.1, TRING.5
- removed net T2: ALU-T.5, PC-T.8, RAM-T.8, REG-T.3, TRING.13, V1.1, V1.9, V5.1
- removed net T3: ALU-T.4, PC-T.7, RAM-T.7, REG-T.2, TRING.12
- removed net T4: ALU-T.3, PC-T.6, RAM-T.6, TRING.11, V1.5
- removed net T5: PC-T.5, RAM-T.5, TRING.10
- removed net T6: ALU-T.2, PC-T.4, RAM-T.4, REG-T.1, TRING.9, V2.3, V2.4
- removed net T7: ALU-T.1, PC-T.3, RAM-T.3, TRING.8
- removed net T8: RAM-T.2, TRING.7, V2.10, V2.11
- removed net T9: PC-T.2, RAM-T.1, TRING.6
- removed net XOA: ALU-OP0.1, INC8.6
- removed net XOV: ALU-OP1.5, INC8.5, PC-OP1.2
- removed net XOX: ALU-OP0.3, INC8.8, REG-OP.4
- removed net XOY: ALU-OP0.2, INC8.7, REG-OP.3
- new net ACP: ALU.2, V15.11
- new net ACP0: IC1.11, V2.3
- new net ACP00: R9.2, V10.1, V2.2
- new net ADD: ALU.6, R15.2, V3.6
- new net ADD0: IC1.17, V2.14
- new net ADD00: R4.2, V15.4, V2.15
- new net AND: ALU.8, R13.2, V3.12
- new net AND0: IC1.19, V2.18
- new net AND00: R1.2, V15.12, V2.19
- new net AOCP: ALU.11, V15.8
- new net AOCP0: IC1.15, V2.8
- new net AOCP00: R6.2, V10.12, V2.9
- new net AOE: ALU.4, R19.2, V4.16
- new net AOE0: IC1.12, V2.4
- new net AOE00: R8.2, V10.4, V2.5
- new net AOOE: ALU.12, R18.2, V4.19
- new net AOOE0: IC1.16, V2.13
- new net AOOE00: R5.2, V15.1, V2.12
- new net C0: IC1.10, IC2.10, IC3.10, IC4.10, RC0.2, V1.3
- new net C1: IC1.9, IC2.9, IC3.9, IC4.9, RC1.2, V1.2
- new net C2: IC1.8, IC2.8, IC3.8, IC4.8, RC2.2, V1.6
- new net C3: IC1.7, IC2.7, IC3.7, IC4.7, RC3.2, V1.7
- new net CP: V2.11, V3.11, V4.11, V5.11, V9.8
- new net EF: FLAG.4, V11.13
- new net FCP: ALU.1, V15.6
- new net FCP0: IC1.13, V2.7
- new net FCP00: R7.2, V10.9, V2.6
- new net GF: FLAG.2, V11.10
- new net INC: V1.5, V6.4, V9.3
- new net IR0: IC1.4, IC2.4, IC3.4, IC4.4, IR.2, RIR0.2, V8.1
- new net IR1: IC1.3, IC2.3, IC3.3, IC4.3, IR.5, RIR1.2, V8.2
- new net IR2: IC1.25, IC2.25, IC3.25, IC4.25, IR.6, RIR2.2, V8.3
- new net IR3: IC1.24, IC2.24, IC3.24, IC4.24, IR.9, RIR3.2
- new net IR4: IC1.21, IC2.21, IC3.21, IC4.21, IR.12, RIR4.2
- new net IR5: IC1.23, IC2.23, IC3.23, IC4.23, IR.15, RIR5.2
- new net IR6: IC1.2, IC2.2, IC3.2, IC4.2, IR.16, RIR6.2
- new net LF: FLAG.6, V11.5
- new net N$100: V12.12, V19.8
- new net N$123: ALU.14
- new net N$13: V14.3, V9.1, V9.2, V9.4, V9.5, V9.9
- new net N$14: V18.2, V19.10, V19.9
- new net N$15: V14.14, V14.2
- new net N$16: NOT.A, R10.1
- new net N$17: R11.1, XOR.A
- new net N$18: IC4.16, V5.13
- new net N$19: OR.A, R12.1
- new net N$20: AND.A, R13.1
- new net N$21: R14.1, SUB.A
- new net N$22: ADD.A, R15.1
- new net N$23: PHCP.A, R16.1
- new net N$24: PLCP.A, R17.1
- new net N$25: AOOE.A, R18.1
- new net N$26: AOE.A, R19.1
- new net N$27: POE.A, R20.1
- new net N$28: PCLR.A, R21.1
- new net N$29: PHOE.A, R22.1
- new net N$3: LC1.A, RC1.1
- new net N$30: PLOE.A, R23.1
- new net N$31: PLD.A, R24.1
- new net N$32: PINC.A, R25.1
- new net N$33: V1.12, V1.14
- new net N$34: V18.4, V19.12
- new net N$35: V17.12, V19.4
- new net N$36: V17.10, V19.1
- new net N$37: V11.12, V17.8
- new net N$38: V11.9, V17.6
- new net N$39: V11.4, V17.4
- new net N$4: LC0.A, RC0.1
- new net N$41: V17.1, V8.15
- new net N$42: V17.3, V8.14
- new net N$43: V17.5, V8.13
- new net N$44: V17.9, V8.12
- new net N$45: V17.11, V8.11
- new net N$46: V17.13, V8.10
- new net N$47: V18.1, V8.9
- new net N$48: V18.3, V8.7
- new net N$49: R26.1, RLD.A
- new net N$5: ACP.A, R1.1
- new net N$50: R27.1, YOE.A
- new net N$51: R28.1, XOE.A
- new net N$52: R29.1, ROE.A
- new net N$53: R30.1, RWE.A
- new net N$54: V13.8, V18.5
- new net N$57: LIR0.A, RIR0.1
- new net N$58: LIR1.A, RIR1.1
- new net N$59: LIR2.A, RIR2.1
- new net N$60: LIR3.A, RIR3.1
- new net N$65: LIR4.A, RIR4.1
- new net N$7: FCP.A, R4.1
- new net N$72: LIR5.A, RIR5.1
- new net N$73: LIR6.A, RIR6.1
- new net N$77: V12.11, V13.5
- new net N$78: V12.8, V13.4
- new net N$79: V12.3, V13.1
- new net N$8: R5.1, XCP.A
- new net N$80: V12.6, V13.2
- new net N$85: V13.3, V13.9
- new net N$86: V13.10, V13.6
- new net N$90: V11.6, V12.1, V12.2
- new net N$91: V11.8, V12.4
- new net N$92: V11.11, V12.5
- new net N$93: V12.9, V19.3
- new net N$94: V12.10, V19.6
- new net N$97: ALU.5
- new net N$98: ALU.3
- new net N$99: V12.13, V19.11
- new net NCLK: V10.10, V10.13, V10.2, V10.5, V15.10, V15.13, V15.2, V15.5, V16.2, V16.5, V6.1, V6.6, V9.12
- new net NG: FLAG.3, V19.5
- new net NOT: ALU.9, R10.2, V3.19
- new net NOT0: IC2.13, V3.7
- new net OCP0: IC3.19, V4.18
- new net OE: IC1.22, IC2.22, IC3.22, IC4.22, V9.6
- new net OF: FLAG.5, V19.2
- new net OR: ALU.10, R12.2, V3.15
- new net OR0: IC2.11, V3.3
- new net OR00: R17.2, V16.1, V3.2
- new net PCLD: C1.1, IR.1, R2.1, S1.1, S1.2, V1.11, V14.11
- new net PCLR: PC.2, R21.2, V4.12
- new net PCLR0: IC3.11, V4.3
- new net PHCP: PC.5, V16.6
- new net PHCP0: IC2.16, V3.13
- new net PHOE: PC.6, R22.2, V4.9
- new net PHOE0: IC2.18, V3.17
- new net PINC: PC.4, R25.2, V4.2
- new net PINC0: IC2.19, V3.18
- new net PLCP: PC.1, V16.3
- new net PLCP0: IC2.15, V3.8
- new net PLD: PC.3, R24.2, V4.5
- new net PLD0: IC3.12, V8.6
- new net PLD1: V18.6, V4.4
- new net PLOE: PC.8, R23.2, V4.6
- new net PLOE0: IC2.17, V3.14
- new net POE: PC.7, R20.2, V4.15
- new net POE0: IC3.13, V4.7
- new net RHCP: RAM.2, V10.6
- new net RHCP0: IC3.16, V4.13
- new net RL: IR.11, V9.11
- new net RLCP: RAM.1, V10.8
- new net RLCP0: IC3.15, V4.8
- new net RLD: R26.2, V5.12, V9.13
- new net ROE: R29.2, RAM.4, V5.5
- new net ROE0: IC3.18, V4.17
- new net RWE: RAM.3, V6.3
- new net RWE0: IC3.17, V4.14
- new net RWE000: R30.2, V5.2, V6.2
- new net SUB: ALU.13, R14.2, V3.9
- new net SUB0: IC1.18, V2.17
- new net SUB00: R3.2, V15.9, V2.16
- new net XCP: REG.1, V15.3
- new net XCP0: IC4.11, V5.3
- new net XOE: R28.2, REG.3, V5.6
- new net XOE0: IC4.12, V5.4
- new net XOR: ALU.7, R11.2, V3.16
- new net XOR0: IC2.12, V3.4
- new net XOR00: R16.2, V16.4, V3.5
- new net YCP: REG.2, V10.11
- new net YCP0: IC4.13, V5.7
- new net YOE: R27.2, REG.4, V5.9
- new net YOE0: IC4.15, V5.8
- new net ZF: FLAG.1, V19.13
- net B0: now also BUSIN.1, IR.3; no longer 0X00.18, 0XFE.18, 0XFF.18, BUS.8, DECODER.3
- net B1: now also BUSIN.2, IR.4; no longer 0X00.17, 0XFE.17, 0XFF.17, BUS.7, DECODER.4
- net B2: now also BUSIN.3, IR.7; no longer 0X00.16, 0XFE.16, 0XFF.16, BUS.6, DECODER.5
- net B3: now also BUSIN.4, IR.8; no longer 0X00.15, 0XFE.15, 0XFF.15, BUS.5, DECODER.6
- net B4: now also BUSIN.5, IR.13; no longer 0X00.14, 0XFE.14, 0XFF.14, BUS.4, DECODER.7
- net B5: now also BUSIN.6, IR.14; no longer 0X00.13, 0XFE.13, 0XFF.13, BUS.3, DECODER.8
- net B6: now also BUSIN.7, IR.17; no longer 0X00.12, 0XFE.12, 0XFF.12, BUS.2, DECODER.9
- net B7: now also BUSIN.8, IR.18; no longer 0X00.11, 0XFE.11, 0XFF.11, BUS.1, DECODER.10
- net CLK: now also CLK.1, V14.5, V6.5, V9.10; no longer ALU-CLK.1, CLK.2, PC-CLK.1, RAM-CLK.1, REG-CLK.1, TRING.2, V1.12, V5.2
- net GND: now also ACP.K, ADD.K, AND.K, AOCP.K, AOE.K, AOOE.K, C1.2, CLK-PS.2, FCP.K, IC1.14, IC1.20, IC1.5, IC1.6, IC2.14, IC2.20, IC2.5, IC2.6, IC3.14, IC3.20, IC3.5, IC3.6, IC4.14, IC4.20, IC4.5, IC4.6, IR.10, LC0.K, LC1.K, LC2.K, LC3.K, LIR0.K, LIR1.K, LIR2.K, LIR3.K, LIR4.K, LIR5.K, LIR6.K, NOT.K, OCP.K, OR.K, PCLR.K, PHCP.K, PHOE.K, PINC.K, PLCP.K, PLD.K, PLOE.K, POE.K, PS.2, RHCP.K, RLCP.K, RLD.K, ROE.K, RWE.K, S1.3, S1.4, SUB.K, V1.1, V1.10, V1.15, V1.4, V1.8, V1.9, V10.7, V11.7, V12.7, V13.7, V14.1, V14.10, V14.15, V14.4, V14.8, V14.9, V15.7, V16.7, V17.7, V18.7, V19.7, V2.10, V3.10, V4.10, V5.10, V6.7, V8.4, V8.5, V8.8, V9.7, XCP.K, XOE.K, XOR.K, YCP.K, YOE.K; no longer 0X00.10, 0X00.2, 0X00.3, 0X00.4, 0X00.5, 0X00.6, 0X00.7, 0X00.8, 0X00.9, 0XFE.10, 0XFE.2, 0XFF.10, ALU-PS.1, C1.-, C2.-, C3.-, C4.-, C5.-, C6.-, C7.-, CLK-PS.1, DECODER.2, PC-PS.1, PS.1, RAM-PS.1, REG-PS.1, TRING.3, V1.7, V2.7, V3.7, V4.7, V5.7
- net HLT: now also HLT.1, IR.19; no longer CLK.1, INC2.1
- net N$1: now also LC3.A, RC3.1; no longer V1.2, V2.12
- net N$10: now also R7.1, RLCP.A; no longer V1.6, V4.5
- net N$11: now also R8.1, RHCP.A; no longer V2.6, V4.2
- net N$12: now also OCP.A, R9.1; no longer V1.8, V4.1
- net N$2: now also LC2.A, RC2.1; no longer V2.5, V2.9, V3.8
- net N$6: now also AOCP.A, R3.1; no longer V5.13, V5.6
- net N$9: now also R6.1, YCP.A; no longer V2.8, V4.4
- net OCP: now also OCP-P.1, V10.3; no longer OCP.1, V5.12
- net VCC: now also CLK-PS.1, IC1.27, IC1.28, IC2.27, IC2.28, IC3.27, IC3.28, IC4.27, IC4.28, IR.20, PS.1, R2.2, V1.16, V10.14, V11.14, V12.14, V13.14, V14.16, V15.14, V16.14, V17.14, V18.14, V19.14, V2.1, V2.20, V3.1, V3.20, V4.1, V4.20, V5.1, V5.20, V6.14, V8.16, V9.14; no longer 0X00.1, 0X00.20, 0XFE.1, 0XFE.20, 0XFE.3, 0XFE.4, 0XFE.5, 0XFE.6, 0XFE.7, 0XFE.8, 0XFE.9, 0XFF.1, 0XFF.2, 0XFF.20, 0XFF.3, 0XFF.4, 0XFF.5, 0XFF.6, 0XFF.7, 0XFF.8, 0XFF.9, ALU-PS.2, C1.+, C2.+, C3.+, C4.+, C5.+, C6.+, C7.+, CLK-PS.2, DECODER.1, PC-PS.2, PS.2, RAM-PS.2, REG-PS.2, TRING.4, V1.14, V2.14, V3.14, V4.14, V5.14
Routing:
- net T2: track 734.4 -> 0.00 mm, vias 9 -> 0
- net T6: track 640.3 -> 0.00 mm, vias 6 -> 0
- net T4: track 625.7 -> 0.00 mm, vias 9 -> 0
- net CLK: track 826.9 -> 216.4 mm, vias 10 -> 2
- net JE: track 586.6 -> 0.00 mm, vias 13 -> 0
- net JG: track 583.9 -> 0.00 mm, vias 13 -> 0
- net JL: track 573.2 -> 0.00 mm, vias 12 -> 0
- net JN: track 567.4 -> 0.00 mm, vias 11 -> 0
- net JNZ: track 562.7 -> 0.00 mm, vias 11 -> 0
- net ADI: track 562.5 -> 0.00 mm, vias 3 -> 0
- net LDAI: track 561.2 -> 0.00 mm, vias 3 -> 0
- net JZ: track 557.3 -> 0.00 mm, vias 11 -> 0
- net LDXI: track 548.5 -> 0.00 mm, vias 6 -> 0
- net RET: track 547.2 -> 0.00 mm, vias 10 -> 0
- net LDYI: track 540.4 -> 0.00 mm, vias 6 -> 0
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Other:
- board size 328.9 x 291.8 mm -> 218.4 x 149.5 mm
