File: Schematics/CTRL/CTRL.sch (EAGLE design)
At the start: 73 parts

Commit message: CTRL v1.1 final version I hope so.
Parts:
- removed ALU-FLAGS: (no value), pinhead:PINHD-2X3
- removed BI, BO, INC1, INC2, INC7, INC8: (no value), pinhead:PINHD-1X8
- removed CLOCK, JP2, OUT, T-CTRL: (no value), pinhead:PINHD-1X2
- removed INC0: (no value), pinhead:PINHD-1X7
- removed INC3, INC4: (no value), pinhead:PINHD-1X5
- removed INC5, INC6: (no value), pinhead:PINHD-1X6
- removed JP1: (no value), pinhead:PINHD-1X11
- removed REGISTER: (no value), pinhead:PINHD-2X2
- added 0X00: 74245N, 74ttl-din:74245N
- added C1, C2, C3: (no value), rcl:CPOL-EUE3.5-8
- added CLK, CLK-PS, JP13: (no value), pinhead:PINHD-1X2
- added DECODER: (no value), pinhead:PINHD-1X11
- added FLAG: (no value), pinhead:PINHD-2X3
- added OP0: (no value), pinhead:PINHD-1X7
- added OP1, OP2, OP5, OP8, OP9: (no value), pinhead:PINHD-1X8
- added OP3, OP4: (no value), pinhead:PINHD-1X5
- added OP6, OP7: (no value), pinhead:PINHD-1X6
- added R2: (no value), rcl:R-EU_0204/7
- added REG: (no value), pinhead:PINHD-2X2
- added S1: (no value), switch-omron:10-XX
- added TRING: (no value), pinhead:PINHD-1X15
- added V51, V54, V60, V63: 7400N, 74ttl-din:7400N
- added V52: 7410N, 74ttl-din:7410N
- added V53: 7430N, 74ttl-din:7430N
- added V55: 7404N, 74ttl-din:7404N
- added V56, V58, V59: 7408N, 74ttl-din:7408N
- added V57, V61, V62: 7432N, 74ttl-din:7432N
- V1: value 7410N -> 7411N; device 74ttl-din:7410N -> 74ttl-din:7411N
- V10: value 7430N -> 7408N; device 74ttl-din:7430N -> 74ttl-din:7408N
- V12: value 7430N -> 7404N; device 74ttl-din:7430N -> 74ttl-din:7404N
- V13, V3, V30, V32, V39, V47, V5: value 7400N -> 7410N; device 74ttl-din:7400N -> 74ttl-din:7410N
- V14, V34, V35, V6, V7: value 7400N -> 7430N; device 74ttl-din:7400N -> 74ttl-din:7430N
- V16, V50: value 7430N -> 7411N; device 74ttl-din:7430N -> 74ttl-din:7411N
- V19, V22: value 7410N -> 7432N; device 74ttl-din:7410N -> 74ttl-din:7432N
- V20, V8: value 7408N -> 7400N; device 74ttl-din:7408N -> 74ttl-din:7400N
- V21: value 7408N -> 7410N; device 74ttl-din:7408N -> 74ttl-din:7410N
- V23: value 7404N -> 7408N; device 74ttl-din:7404N -> 74ttl-din:7408N
- V24, V42: value 7430N -> 7410N; device 74ttl-din:7430N -> 74ttl-din:7410N
- V25, V9: value 7430N -> 7432N; device 74ttl-din:7430N -> 74ttl-din:7432N
- V26: value 7410N -> 7404N; device 74ttl-din:7410N -> 74ttl-din:7404N
- V27, V44: value 7410N -> 7408N; device 74ttl-din:7410N -> 74ttl-din:7408N
- V31, V37: value 7400N -> 7411N; device 74ttl-din:7400N -> 74ttl-din:7411N
- V33: value 7410N -> 7430N; device 74ttl-din:7410N -> 74ttl-din:7430N
- V36: value 7408N -> 7432N; device 74ttl-din:7408N -> 74ttl-din:7432N
- V4, V40, V45: value 7400N -> 7404N; device 74ttl-din:7400N -> 74ttl-din:7404N
- V41: value 7410N -> 7400N; device 74ttl-din:7410N -> 74ttl-din:7400N
- V43: value 7430N -> 7400N; device 74ttl-din:7430N -> 74ttl-din:7400N
Connections:
- net SL-OE renamed SL
- net SR-OE renamed SR
- removed net !ZERO: V20/3.A, V23/5.Y
- removed net ACC-CP: ALU.2, V48/1.Y, V48/2.Y
- removed net ACC-OE: ALU.4, V47/1.Y
- removed net ADD-OE: ALU.6, V32/1.Y, V32/2.Y, V32/3.Y, V34/2.Y, V34/3.Y, V35/1.Y
- removed net EQUIL: ALU-FLAGS.4, V21/3.A
- removed net FE: 0XFE1.!G
- removed net FF: 0XFF1.!G
- removed net GREATER: ALU-FLAGS.2, V21/2.A
- removed net LESS: ALU-FLAGS.6, V21/1.A
- removed net NEGATIVE: ALU-FLAGS.3, V20/4.A
- removed net O0: 0XFE1.B1, 0XFF1.B1, BO.8
- removed net O1: 0XFE1.B2, 0XFF1.B2, BO.7
- removed net O2: 0XFE1.B3, 0XFF1.B3, BO.6
- removed net O3: 0XFE1.B4, 0XFF1.B4, BO.5
- removed net O4: 0XFE1.B5, 0XFF1.B5, BO.4
- removed net O5: 0XFE1.B6, 0XFF1.B6, BO.3
- removed net O6: 0XFE1.B7, 0XFF1.B7, BO.2
- removed net O7: 0XFE1.B8, 0XFF1.B8, BO.1
- removed net OCP: OUT.1, OUT.2
- removed net OE: RAM.4, V27/3.Y, V28/3.Y, V28/4.Y, V29/2.Y
- removed net OUT: ALU.12, V44/3.Y, V45/1.Y, V45/3.Y
- removed net OUT-CP: ALU.11, V41/1.Y, V41/2.Y, V44/2.Y
- removed net OVERFLOW: ALU-FLAGS.5
- removed net PC-OEH: V14/3.Y
- removed net PC-OEL: V14/2.Y
- removed net RAM-HCP: RAM.2, V22/2.Y, V26/3.Y
- removed net RAM-LCP: RAM.1, V22/1.Y, V22/3.Y
- removed net T-CLR: T-CTRL.2
- removed net WE: RAM.3, V28/1.Y, V28/2.Y
- removed net ZERO: ALU-FLAGS.1, V20/2.A, V23/5.A
- new net 0X00: 0X001.!G, V28/1.Y
- new net 0XFE: 0XFE1.!G, V56/2.Y
- new net 0XFF: 0XFF1.!G, V56/1.Y
- new net ACP: ALU.2, V31/1.Y
- new net ADD: ALU.6, V37/1.Y
- new net AOCP: ALU.11, V44/4.Y
- new net AOE: ALU.4, V31/3.Y
- new net AOOE: ALU.12, V50/1.Y
- new net CLK-HLT: CLK.1
- new net EQ: FLAG.4, V59/1.A
- new net GD: FLAG.2, V58/4.A
- new net IRCP: DECODER.11, V60/3.Y
- new net JMP: V11/4.B, V13/2.B, V13/3.A, V151.Y, V19/4.B, V23/1.B, V23/3.A, V23/4.A, V25/1.A, V25/2.B
- new net L1: V25/3.B, V25/4.Y, V36/3.A
- new net L2: V46/3.Y, V47/1.C, V51/1.B
- new net LD: FLAG.6, V58/3.A
- new net N$100: V38/1.B, V39/1.Y
- new net N$101: V40/3.Y, V41/1.B
- new net N$102: V37/1.A, V38/1.Y
- new net N$103: V37/1.B, V38/2.Y
- new net N$104: V37/1.C, V38/3.Y
- new net N$105: V43/4.Y, V44/1.B
- new net N$106: V40/6.Y, V43/2.B
- new net N$107: V40/4.Y, V41/2.B
- new net N$108: V37/2.C, V41/2.Y
- new net N$109: V37/2.B, V41/1.Y
- new net N$110: V37/2.A, V38/4.Y
- new net N$111: V42/1.Y, V43/1.B
- new net N$112: V44/3.A, V47/1.Y
- new net N$113: V44/3.B, V47/2.Y
- new net N$114: V44/3.Y, V44/4.A
- new net N$115: V44/4.B, V48/2.Y
- new net N$116: V42/3.Y, V46/2.B
- new net N$117: V43/4.B, V45/1.Y
- new net N$118: V36/3.B, V491.Y
- new net N$119: V42/2.Y, V43/3.B
- new net N$120: V54/2.Y, V56/2.B
- new net N$121: V45/2.Y, V46/1.B
- new net N$122: V44/2.B, V46/1.Y
- new net N$123: V44/2.A, V46/2.Y
- new net N$124: V50/1.A, V51/1.Y
- new net N$125: V46/4.Y, V50/1.B
- new net N$126: V52/2.Y, V56/2.A
- new net N$127: V48/3.Y, V50/1.C
- new net N$128: V45/3.A, V50/3.Y
- new net N$129: V45/3.Y, V50/2.C
- new net N$130: V52/1.Y, V56/1.B
- new net N$131: V36/2.A, V47/3.Y
- new net N$132: V36/2.B, V48/1.Y
- new net N$133: V36/2.Y, V46/4.A, V47/2.C
- new net N$134: V57/1.Y, V61/1.A
- new net N$135: V45/6.A, V50/2.Y
- new net N$136: V36/3.Y, V48/2.C, V48/3.A, V48/3.B
- new net N$137: V54/3.B, V61/2.Y
- new net N$138: V24/3.Y, V28/1.B
- new net N$139: V54/3.Y, V56/3.B
- new net N$140: V57/4.B, V60/1.Y
- new net N$141: V56/4.Y, V57/1.A
- new net N$142: V57/1.B, V58/1.Y
- new net N$143: V55/1.Y, V58/1.A
- new net N$144: V55/2.Y, V58/1.B
- new net N$145: V57/2.Y, V61/1.B
- new net N$146: V22/4.B, V62/1.Y
- new net N$147: V40/5.Y, V41/3.B
- new net N$148: V57/3.Y, V57/4.A
- new net N$149: V55/3.Y, V58/2.B
- new net N$150: V61/1.Y, V61/2.A
- new net N$151: V55/4.Y, V58/3.B
- new net N$152: V57/4.Y, V61/2.B
- new net N$153: V55/5.Y, V58/4.B
- new net N$154: V23/2.A, V63/1.Y
- new net N$155: V55/6.Y, V59/1.B
- new net N$156: V25/1.B, V25/2.A, V26/1.Y
- new net N$158: V57/2.A, V58/2.Y
- new net N$160: V57/2.B, V58/3.Y
- new net N$162: V57/3.A, V58/4.Y
- new net N$164: V57/3.B, V59/1.Y
- new net N$44: V11/3.A, V17/3.Y
- new net N$51: V16/3.Y, V22/3.B
- new net N$53: V22/3.Y, V22/4.A
- new net N$57: V10/4.A, V20/1.Y
- new net N$60: V21/3.Y, V23/2.B
- new net N$61: V24/1.C, V25/1.Y
- new net N$62: V28/2.B, V30/2.Y
- new net N$63: V24/2.C, V25/2.Y
- new net N$64: V28/2.A, V30/1.Y
- new net N$65: V12/4.A, V23/4.Y
- new net N$66: V12/5.A, V23/3.Y
- new net N$67: V28/2.Y, V29/3.C
- new net N$68: V54/4.Y, V56/4.B
- new net N$69: V29/1.C, V29/2.Y
- new net N$70: V26/3.Y, V30/3.C
- new net N$71: V25/4.B, V32/3.Y
- new net N$72: V29/1.Y, V31/2.A
- new net N$73: V29/3.Y, V31/2.B
- new net N$74: V25/4.A, V341.Y
- new net N$75: V30/3.Y, V31/2.C
- new net N$76: V28/3.Y, V32/1.C
- new net N$77: V52/3.Y, V56/3.A
- new net N$78: V25/3.A, V331.Y
- new net N$79: V31/1.B, V32/1.Y
- new net N$80: V25/3.Y, V32/2.C
- new net N$81: V31/1.A, V31/2.Y
- new net N$82: V26/6.A, V27/3.Y
- new net N$83: V31/1.C, V32/2.Y
- new net N$84: V26/4.Y, V28/4.B
- new net N$85: V351.Y, V36/1.A
- new net N$86: V28/4.Y, V31/3.A
- new net N$87: V26/6.Y, V31/3.B, V31/3.C
- new net N$88: V26/5.Y, V36/1.B
- new net N$89: V26/5.A, V27/2.Y
- new net N$90: V27/3.A, V36/1.Y
- new net N$91: V37/3.B, V37/3.C, V41/3.Y
- new net N$92: V37/3.A, V41/4.Y
- new net N$93: V43/3.Y, V44/1.A
- new net N$94: V39/3.Y, V41/4.B
- new net N$95: V27/4.A, V43/1.Y
- new net N$96: V38/3.B, V40/2.Y
- new net N$97: V38/4.B, V39/2.Y
- new net N$98: V38/2.B, V40/1.Y
- new net N$99: V27/4.B, V43/2.Y
- new net NG: FLAG.3, V58/2.A
- new net OF: FLAG.5
- new net RHCP: RAM.2, V16/1.Y
- new net RLCP: RAM.1, V1/3.Y
- new net ROE: RAM.4, V10/4.Y
- new net RWE: RAM.3, V10/3.Y
- new net T0: TRING.15, V62/1.B
- new net T1: TRING.14, V60/3.A, V63/1.A
- new net TCLR: TRING.1
- new net ZF: FLAG.1, V55/2.A, V56/4.A
- net ADA: now also OP3.3, V331.D, V351.C, V39/1.C; no longer INC3.3, V33/1.C, V421.C, V47/2.A
- net ADI: now also OP3.2, V141.D, V21/1.A, V28/3.B, V40/2.A, V46/3.B; no longer INC3.2, V121.D, V26/1.A, V27/1.A, V34/1.A, V34/1.B, V45/2.A, V91.E
- net ADV: now also OP3.1, V181.B, V30/1.A, V40/1.A, V47/3.A; no longer INC3.1, V32/4.A, V32/4.B, V41/3.A, V91.F
- net ADX: now also OP3.5, V331.B, V39/1.A, V491.A, V61.C; no longer INC3.5, V33/1.A, V4/1.A, V421.A
- net ADY: now also OP3.4, V331.C, V39/1.B, V71.C; no longer INC3.4, V33/1.B, V421.B, V6/3.A
- net ANA: now also OP8.6, V341.B, V351.G, V39/3.C; no longer INC7.6
- net AND: now also V37/3.Y; no longer V37/1.Y, V38/3.Y
- net ANV: now also OP8.5, V181.G, V30/1.C, V40/5.A, V47/3.C; no longer INC7.5, V101.G, V38/4.A, V38/4.B, V41/3.C
- net ANX: now also OP8.8, V331.H, V39/3.A, V61.G; no longer INC7.8, V37/2.A, V4/3.A, V421.G
- net ANY: now also OP8.7, V341.A, V39/3.B, V71.G; no longer INC7.7, V37/2.B, V421.H, V501.A, V7/1.A
- net B0: now also 0X001.B1, 0XFE1.B1, 0XFF1.B1, DECODER.3, OP5.8; no longer BI.8
- net B1: now also 0X001.B2, 0XFE1.B2, 0XFF1.B2, DECODER.4, OP5.7; no longer BI.7
- net B2: now also 0X001.B3, 0XFE1.B3, 0XFF1.B3, DECODER.5, OP5.6; no longer BI.6
- net B3: now also 0X001.B4, 0XFE1.B4, 0XFF1.B4, DECODER.6, OP5.5; no longer BI.5
- net B4: now also 0X001.B5, 0XFE1.B5, 0XFF1.B5, DECODER.7, OP5.4; no longer BI.4
- net B5: now also 0X001.B6, 0XFE1.B6, 0XFF1.B6, DECODER.8, OP5.3; no longer BI.3
- net B6: now also 0X001.B7, 0XFE1.B7, 0XFF1.B7, DECODER.9, OP5.2; no longer BI.2
- net B7: now also 0X001.B8, 0XFE1.B8, 0XFF1.B8, DECODER.10, OP5.1; no longer BI.1
- net CALL: now also OP1.4, V531.A, V60/1.A, V60/1.B; no longer INC1.4, V11/2.A, V161.A, V181.A, V241.A, V251.A
- net CLA: now also OP0.4, V24/3.A, V29/2.A; no longer INC0.4, V46/4.A, V46/4.B
- net CLK: now also CLK.2, TRING.2, V13/1.A, V13/2.A, V13/3.C, V17/1.C, V17/2.A, V2/1.A, V2/3.A, V24/1.B, V24/2.B, V29/1.B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; no longer CLOCK.2, T-CTRL.1, V1/1.B, V1/3.B, V17/1.B, V17/2.B, V19/1.B, V19/2.B, V2/2.B, V2/3.B, V22/1.B, V22/2.B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
- net CLX: now also OP0.6, V2/2.A, V24/3.B; no longer INC0.6, V1/2.A
- net CLY: now also OP0.5, V24/3.C, V3/3.A; no longer INC0.5, V2/1.A
- net CMA: now also OP1.6, V351.B, V50/3.C; no longer INC1.6
- net CMV: now also OP1.5, V181.A; no longer INC1.5, V46/3.A, V46/3.B, V91.A
- net CMX: now also OP1.8, V50/3.A, V61.B; no longer INC1.8, V3/4.B, V46/1.A
- net CMY: now also OP1.7, V50/3.B, V71.B; no longer INC1.7, V46/1.B, V6/2.B
- net FCP: now also V45/6.Y; no longer V45/4.Y, V46/2.Y
- net GND: now also 0X00/-UB.-UB, 0X001.A1, 0X001.A2, 0X001.A3, 0X001.A4, 0X001.A5, 0X001.A6, 0X001.A7, 0X001.A8, C1.-, C2.-, C3.-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; no longer JP2.1
- net HLT: now also OP2.1; no longer CLOCK.1, INC2.1
- net JE: now also OP2.3, V531.F, V55/6.A; no longer INC2.3, V13/1.A, V13/1.B, V161.G, V161.H, V21/3.B, V241.G, V251.G
- net JG: now also OP2.4, V531.E, V55/5.A; no longer INC2.4, V11/4.B, V161.F, V21/2.B, V241.F, V251.F
- net JL: now also OP2.5, V531.G, V531.H, V55/4.A; no longer INC2.5, V11/4.A, V161.E, V21/1.B, V241.E, V251.E
- net JN: now also OP2.6, V531.D, V55/3.A; no longer INC2.6, V11/3.B, V161.D, V20/4.B, V241.D, V251.D
- net JNZ: now also OP2.7, V531.C, V55/1.A; no longer INC2.7, V11/3.A, V161.C, V20/3.B, V241.C, V251.C
- net JZ: now also OP2.8, V531.B, V54/4.A, V54/4.B; no longer INC2.8, V11/2.B, V161.B, V20/2.B, V241.B, V251.B
- net LDA: now also OP6.4, V181.F, V331.A; no longer INC5.4, V101.C, V491.A
- net LDAI: now also OP6.1, V141.H, V21/2.B, V21/2.C, V26/3.A; no longer INC5.1, V101.F, V121.H, V26/2.B, V26/2.C, V27/2.B, V27/2.C, V29/3.C
- net LDX: now also OP6.6, V181.D, V4/1.A; no longer INC5.6, V101.A
- net LDXI: now also OP6.3, V141.F, V21/1.C, V4/2.A; no longer INC5.3, V101.D, V121.F, V26/1.C, V27/1.C, V29/3.A, V3/1.A, V3/1.B
- net LDY: now also OP6.5, V181.E, V4/3.A; no longer INC5.5, V101.B
- net LDYI: now also OP6.2, V141.G, V21/2.A, V4/4.A; no longer INC5.2, V101.E, V121.G, V26/2.A, V27/2.A, V29/3.B, V3/2.A, V3/2.B
- net MAX: now also OP7.2, V29/2.B, V61.F; no longer INC6.2, V4/2.A
- net MAY: now also OP7.1, V29/2.C, V71.F; no longer INC6.1, V6/4.B
- net MXA: now also OP7.5, V2/2.C, V351.E; no longer INC6.5, V1/2.C
- net MXY: now also OP7.6, V2/2.B, V71.E; no longer INC6.6, V1/2.B, V6/4.A
- net MYA: now also OP7.3, V3/3.C, V351.F; no longer INC6.3, V2/1.C
- net MYX: now also OP7.4, V3/3.B, V61.E; no longer INC6.4, V2/1.B, V4/2.B
- net N$1: now also V10/2.A, V11/2.Y; no longer V23/1.Y, V23/2.A
- net N$10: now also V11/2.B, V9/2.Y; no longer V101.Y, V11/1.Y, V13/2.A, V8/1.B, V91.Y
- net N$11: now also V8/2.Y, V9/2.B; no longer V5/1.B, V5/2.Y
- net N$12: now also V2/1.C, V2/2.Y; no longer V121.Y, V13/3.A, V8/2.B
- net N$13: now also V71.Y, V9/2.A; no longer V11/2.Y, V11/3.Y, V11/4.Y, V13/1.Y, V13/4.A, V14/1.A, V8/3.B, V8/4.A
- net N$14: now also V3/2.C, V3/3.Y; no longer V17/2.C, V181.Y, V19/2.C, V31/1.A
- net N$15: now also V1/1.A, V2/1.Y; no longer V2/3.C, V3/2.Y
- net N$16: now also V1/1.B, V2/3.Y; no longer V5/3.B, V5/4.Y
- net N$17: now also V1/1.C, V3/1.Y; no longer V19/1.C, V19/3.Y
- net N$18: now also V5/3.B, V9/3.Y; no longer V14/2.B, V161.Y
- net N$19: now also V12/1.Y, V5/3.C; no longer V181.G, V181.H, V21/3.Y
- net N$2: now also V1/2.A, V3/2.Y; no longer JP1.10, V23/3.A
- net N$20: now also V13/1.C, V141.Y, V17/1.A, V19/4.A; no longer V17/1.C, V17/3.Y
- net N$21: now also V1/3.B, V13/1.Y; no longer V181.F, V21/2.Y
- net N$22: now also V4/3.Y, V5/1.C; no longer V181.E, V21/1.Y
- net N$23: now also V1/3.C, V13/2.Y; no longer V181.D, V20/4.Y
- net N$24: now also V8/1.Y, V9/1.B; no longer V181.C, V20/3.Y
- net N$25: now also V61.Y, V9/1.A; no longer V181.B, V20/2.Y
- net N$26: now also V10/1.A, V8/4.Y; no longer V22/3.C, V26/1.Y, V26/2.Y
- net N$27: now also V10/1.B, V8/3.Y; no longer V14/3.B, V151.Y
- net N$28: now also V4/5.Y, V8/3.B; no longer V26/3.C, V27/1.Y, V27/2.Y
- net N$29: now also V13/2.C, V9/4.Y; no longer V22/1.C, V241.Y, V28/1.A
- net N$3: now also V1/2.B, V5/1.Y; no longer V1/1.C, V1/2.Y
- net N$30: now also V8/4.B, V9/1.Y; no longer V22/2.C, V251.Y, V28/2.A
- net N$31: now also V11/1.B, V4/6.Y; no longer V34/3.B, V34/4.Y, V36/2.B
- net N$32: now also V52/1.C, V52/2.A, V531.Y; no longer V29/2.B, V29/2.C, V29/3.Y
- net N$33: now also V12/2.Y, V17/2.C; no longer V32/3.B, V34/1.Y
- net N$34: now also V11/4.A, V19/1.Y; no longer V28/3.B, V28/4.A, V29/1.Y
- net N$35: now also V19/2.B, V21/2.Y; no longer V27/3.B, V27/3.C, V30/1.Y, V30/2.Y
- net N$36: now also ALU.14; no longer V32/2.B, V32/4.Y
- net N$37: now also V20/3.Y, V22/1.B; no longer V33/2.Y, V34/2.B, V36/1.A
- net N$38: now also V16/1.B, V17/1.Y; no longer V32/1.B, V33/1.Y
- net N$39: now also V16/1.C, V17/2.Y; no longer V37/1.B, V37/2.Y
- net N$4: now also V1/2.C, V5/2.Y; no longer V1/3.C, V2/1.Y
- net N$40: now also V13/3.Y, V16/1.A; no longer V35/1.B, V35/2.B, V35/3.Y
- net N$41: now also V19/2.A, V21/1.Y; no longer V33/3.Y, V35/4.B
- net N$42: now also V10/3.B, V11/4.Y; no longer V41/2.C, V41/3.Y, V44/1.Y, V45/3.A
- net N$43: now also V10/3.A, V11/3.Y; no longer V38/3.B, V38/4.Y
- net N$45: now also V181.Y, V22/1.A; no longer V46/2.B, V46/3.Y
- net N$46: now also V22/1.Y, V22/2.A; no longer V45/4.B, V46/1.Y
- net N$47: now also V16/3.A, V19/4.Y, V21/3.A, V22/2.B; no longer V40/1.B, V40/2.Y
- net N$48: now also V16/2.C, V20/4.B, V22/2.Y; no longer V37/3.B, V37/4.Y
- net N$49: now also V23/1.Y, V62/1.A; no longer V38/1.B, V38/2.Y
- net N$5: now also V4/4.Y, V5/2.C; no longer V6/1.B, V6/2.Y, V6/3.Y, V6/4.Y, V7/1.Y, V7/2.Y
- net N$50: now also V16/2.Y, V22/3.A; no longer V41/1.C, V421.Y, V431.Y, V45/1.A
- net N$52: now also V19/2.Y, V20/2.B; no longer V46/4.Y, V48/1.C
- net N$54: now also V12/3.Y, V20/1.B; no longer V48/2.C, V491.Y, V501.Y
- net N$55: now also V19/3.Y, V20/1.A; no longer V44/2.C, V44/3.C, V45/2.Y
- net N$56: now also V10/4.B, V20/2.Y; no longer V39/1.B, V39/2.Y
- net N$58: now also V54/1.Y, V56/1.A; no longer V47/1.B, V47/2.Y, V47/3.Y
- net N$59: now also V20/4.Y, V63/1.B; no longer V39/3.B, V39/4.Y
- net N$6: now also V3/1.C, V4/2.Y; no longer JP1.11, V23/1.A
- net N$7: now also V1/3.A, V5/3.Y; no longer V2/2.C, V3/1.Y
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
Commit message: Final version of CTRL-bus. last brd is bus.
Parts:
- removed ALU: (no value), pinhead:PINHD-2X7
- removed FLAG: (no value), pinhead:PINHD-2X3
- removed PC: (no value), pinhead:PINHD-2X4
- removed R2: (no value), rcl:R-EU_0204/7
- removed RAM, REG: (no value), pinhead:PINHD-2X2
- removed S1: (no value), switch-omron:10-XX
- removed V10, V23, V27, V44, V56, V58, V59: 7408N, 74ttl-din:7408N
- removed V11, V20, V28, V38, V41, V43, V46, V51, V54, V60, V63, V8: 7400N, 74ttl-din:7400N
- removed V12, V26, V40, V45, V55: 7404N, 74ttl-din:7404N
- removed V13, V17, V21, V24, V29, V30, V32, V39, V42, V47, V48, V5, V52: 7410N, 74ttl-din:7410N
- removed V14, V15, V18, V33, V34, V35, V49, V53, V6, V7: 7430N, 74ttl-din:7430N
- removed V16, V31, V37, V50: 7411N, 74ttl-din:7411N
- removed V19, V22, V25, V36, V57, V61, V62, V9: 7432N, 74ttl-din:7432N
- added ALU-CLK, PC-CLK, PC-CLR, RAM-CLK, REG-CLK: (no value), pinhead:PINHD-1X1
- added ALU-OP0, REG-OP: (no value), pinhead:PINHD-1X30
- added ALU-OP1, ALU-T: (no value), pinhead:PINHD-1X5
- added ALU-PS, PC-OP1, PC-PS, RAM-PS, REG-PS: (no value), pinhead:PINHD-1X2
- added C4, C5, C6, C7: (no value), rcl:CPOL-EUE2.5-6
- added PC-OP0: (no value), pinhead:PINHD-1X24
- added PC-T: (no value), pinhead:PINHD-1X10
- added RAM-OP: (no value), pinhead:PINHD-1X16
- added RAM-T: (no value), pinhead:PINHD-1X8
- added REG-T: (no value), pinhead:PINHD-1X3
- C1, C2, C3: device rcl:CPOL-EUE3.5-8 -> rcl:CPOL-EUE2.5-6
- V1: value 7411N -> 7400N; device 74ttl-din:7411N -> 74ttl-din:7400N
- V3: value 7410N -> 7430N; device 74ttl-din:7410N -> 74ttl-din:7430N
- V4: value 7404N -> 7408N; device 74ttl-din:7404N -> 74ttl-din:7408N
- renumbered JP13 to PS, OP0 to INC0, OP1 to INC1, OP2 to INC2, OP3 to INC3, OP4 to INC4, OP5 to BUS, OP6 to INC5, OP7 to INC6, OP8 to INC7, OP9 to INC8
Connections:
- removed net ACP: ALU.2, V31/1.Y
- removed net ADD: ALU.6, V37/1.Y
- removed net AND: ALU.8, V37/3.Y
- removed net AOCP: ALU.11, V44/4.Y
- removed net AOE: ALU.4, V31/3.Y
- removed net AOOE: ALU.12, V50/1.Y
- removed net CLK-HLT: CLK.1
- removed net EQ: FLAG.4, V59/1.A
- removed net FCP: ALU.1, V45/6.Y
- removed net GD: FLAG.2, V58/4.A
- removed net JMP: V11/4.B, V13/2.B, V13/3.A, V151.Y, V19/4.B, V23/1.B, V23/3.A, V23/4.A, V25/1.A, V25/2.B
- removed net L1: V25/3.B, V25/4.Y, V36/3.A
- removed net L2: V46/3.Y, V47/1.C, V51/1.B
- removed net LD: FLAG.6, V58/3.A
- removed net N$100: V38/1.B, V39/1.Y
- removed net N$101: V40/3.Y, V41/1.B
- removed net N$102: V37/1.A, V38/1.Y
- removed net N$103: V37/1.B, V38/2.Y
- removed net N$104: V37/1.C, V38/3.Y
- removed net N$105: V43/4.Y, V44/1.B
- removed net N$106: V40/6.Y, V43/2.B
- removed net N$107: V40/4.Y, V41/2.B
- removed net N$108: V37/2.C, V41/2.Y
- removed net N$109: V37/2.B, V41/1.Y
- removed net N$110: V37/2.A, V38/4.Y
- removed net N$111: V42/1.Y, V43/1.B
- removed net N$112: V44/3.A, V47/1.Y
- removed net N$113: V44/3.B, V47/2.Y
- removed net N$114: V44/3.Y, V44/4.A
- removed net N$115: V44/4.B, V48/2.Y
- removed net N$116: V42/3.Y, V46/2.B
- removed net N$117: V43/4.B, V45/1.Y
- removed net N$118: V36/3.B, V491.Y
- removed net N$119: V42/2.Y, V43/3.B
- removed net N$120: V54/2.Y, V56/2.B
- removed net N$121: V45/2.Y, V46/1.B
- removed net N$122: V44/2.B, V46/1.Y
- removed net N$123: V44/2.A, V46/2.Y
- removed net N$124: V50/1.A, V51/1.Y
- removed net N$125: V46/4.Y, V50/1.B
- removed net N$126: V52/2.Y, V56/2.A
- removed net N$127: V48/3.Y, V50/1.C
- removed net N$128: V45/3.A, V50/3.Y
- removed net N$129: V45/3.Y, V50/2.C
- removed net N$13: V71.Y, V9/2.A
- removed net N$130: V52/1.Y, V56/1.B
- removed net N$131: V36/2.A, V47/3.Y
- removed net N$132: V36/2.B, V48/1.Y
- removed net N$133: V36/2.Y, V46/4.A, V47/2.C
- removed net N$134: V57/1.Y, V61/1.A
- removed net N$135: V45/6.A, V50/2.Y
- removed net N$136: V36/3.Y, V48/2.C, V48/3.A, V48/3.B
- removed net N$137: V54/3.B, V61/2.Y
- removed net N$138: V24/3.Y, V28/1.B
- removed net N$139: V54/3.Y, V56/3.B
- removed net N$14: V3/2.C, V3/3.Y
- removed net N$140: V57/4.B, V60/1.Y
- removed net N$141: V56/4.Y, V57/1.A
- removed net N$142: V57/1.B, V58/1.Y
- removed net N$143: V55/1.Y, V58/1.A
- removed net N$144: V55/2.Y, V58/1.B
- removed net N$145: V57/2.Y, V61/1.B
- removed net N$146: V22/4.B, V62/1.Y
- removed net N$147: V40/5.Y, V41/3.B
- removed net N$148: V57/3.Y, V57/4.A
- removed net N$149: V55/3.Y, V58/2.B
- removed net N$15: V1/1.A, V2/1.Y
- removed net N$150: V61/1.Y, V61/2.A
- removed net N$151: V55/4.Y, V58/3.B
- removed net N$152: V57/4.Y, V61/2.B
- removed net N$153: V55/5.Y, V58/4.B
- removed net N$154: V23/2.A, V63/1.Y
- removed net N$155: V55/6.Y, V59/1.B
- removed net N$156: V25/1.B, V25/2.A, V26/1.Y
- removed net N$158: V57/2.A, V58/2.Y
- removed net N$16: V1/1.B, V2/3.Y
- removed net N$160: V57/2.B, V58/3.Y
- removed net N$162: V57/3.A, V58/4.Y
- removed net N$164: V57/3.B, V59/1.Y
- removed net N$17: V1/1.C, V3/1.Y
- removed net N$18: V5/3.B, V9/3.Y
- removed net N$19: V12/1.Y, V5/3.C
- removed net N$20: V13/1.C, V141.Y, V17/1.A, V19/4.A
- removed net N$21: V1/3.B, V13/1.Y
- removed net N$22: V4/3.Y, V5/1.C
- removed net N$23: V1/3.C, V13/2.Y
- removed net N$24: V8/1.Y, V9/1.B
- removed net N$25: V61.Y, V9/1.A
- removed net N$26: V10/1.A, V8/4.Y
- removed net N$27: V10/1.B, V8/3.Y
- removed net N$28: V4/5.Y, V8/3.B
- removed net N$29: V13/2.C, V9/4.Y
- removed net N$3: V1/2.B, V5/1.Y
- removed net N$30: V8/4.B, V9/1.Y
- removed net N$31: V11/1.B, V4/6.Y
- removed net N$32: V52/1.C, V52/2.A, V531.Y
- removed net N$33: V12/2.Y, V17/2.C
- removed net N$34: V11/4.A, V19/1.Y
- removed net N$35: V19/2.B, V21/2.Y
- removed net N$36: ALU.14
- removed net N$37: V20/3.Y, V22/1.B
- removed net N$38: V16/1.B, V17/1.Y
- removed net N$39: V16/1.C, V17/2.Y
- removed net N$4: V1/2.C, V5/2.Y
- removed net N$40: V13/3.Y, V16/1.A
- removed net N$41: V19/2.A, V21/1.Y
- removed net N$42: V10/3.B, V11/4.Y
- removed net N$43: V10/3.A, V11/3.Y
- removed net N$44: V11/3.A, V17/3.Y
- removed net N$45: V181.Y, V22/1.A
- removed net N$46: V22/1.Y, V22/2.A
- removed net N$47: V16/3.A, V19/4.Y, V21/3.A, V22/2.B
- removed net N$48: V16/2.C, V20/4.B, V22/2.Y
- removed net N$49: V23/1.Y, V62/1.A
- removed net N$5: V4/4.Y, V5/2.C
- removed net N$50: V16/2.Y, V22/3.A
- removed net N$51: V16/3.Y, V22/3.B
- removed net N$52: V19/2.Y, V20/2.B
- removed net N$53: V22/3.Y, V22/4.A
- removed net N$54: V12/3.Y, V20/1.B
- removed net N$55: V19/3.Y, V20/1.A
- removed net N$56: V10/4.B, V20/2.Y
- removed net N$57: V10/4.A, V20/1.Y
- removed net N$58: V54/1.Y, V56/1.A
- removed net N$59: V20/4.Y, V63/1.B
- removed net N$6: V3/1.C, V4/2.Y
- removed net N$60: V21/3.Y, V23/2.B
- removed net N$61: V24/1.C, V25/1.Y
- removed net N$62: V28/2.B, V30/2.Y
- removed net N$63: V24/2.C, V25/2.Y
- removed net N$64: V28/2.A, V30/1.Y
- removed net N$65: V12/4.A, V23/4.Y
- removed net N$66: V12/5.A, V23/3.Y
- removed net N$67: V28/2.Y, V29/3.C
- removed net N$68: V54/4.Y, V56/4.B
- removed net N$69: V29/1.C, V29/2.Y
- removed net N$7: V1/3.A, V5/3.Y
- removed net N$70: V26/3.Y, V30/3.C
- removed net N$71: V25/4.B, V32/3.Y
- removed net N$72: V29/1.Y, V31/2.A
- removed net N$73: V29/3.Y, V31/2.B
- removed net N$74: V25/4.A, V341.Y
- removed net N$75: V30/3.Y, V31/2.C
- removed net N$76: V28/3.Y, V32/1.C
- removed net N$77: V52/3.Y, V56/3.A
- removed net N$78: V25/3.A, V331.Y
- removed net N$79: V31/1.B, V32/1.Y
- removed net N$8: V10/2.B, V11/1.Y
- removed net N$80: V25/3.Y, V32/2.C
- removed net N$81: V31/1.A, V31/2.Y
- removed net N$82: V26/6.A, V27/3.Y
- removed net N$83: V31/1.C, V32/2.Y
- removed net N$84: V26/4.Y, V28/4.B
- removed net N$85: V351.Y, V36/1.A
- removed net N$86: V28/4.Y, V31/3.A
- removed net N$87: V26/6.Y, V31/3.B, V31/3.C
- removed net N$88: V26/5.Y, V36/1.B
- removed net N$89: V26/5.A, V27/2.Y
- removed net N$90: V27/3.A, V36/1.Y
- removed net N$91: V37/3.B, V37/3.C, V41/3.Y
- removed net N$92: V37/3.A, V41/4.Y
- removed net N$93: V43/3.Y, V44/1.A
- removed net N$94: V39/3.Y, V41/4.B
- removed net N$95: V27/4.A, V43/1.Y
- removed net N$96: V38/3.B, V40/2.Y
- removed net N$97: V38/4.B, V39/2.Y
- removed net N$98: V38/2.B, V40/1.Y
- removed net N$99: V27/4.B, V43/2.Y
- removed net NG: FLAG.3, V58/2.A
- removed net NOT: ALU.9, V44/1.Y
- removed net OF: FLAG.5
- removed net OR: ALU.10, V27/4.Y
- removed net PC-CLR: PC.2, R2.2, S1.P, S1.P1
- removed net PC-HCP: PC.5, V24/2.Y
- removed net PC-HOE: PC.6, V12/4.Y
- removed net PC-INC: PC.4, V22/4.Y
- removed net PC-LCP: PC.1, V24/1.Y
- removed net PC-LD: PC.3, V56/3.Y
- removed net PC-LOE: PC.8, V12/5.Y
- removed net PC-OE: PC.7, V23/2.Y
- removed net RHCP: RAM.2, V16/1.Y
- removed net RLCP: RAM.1, V1/3.Y
- removed net ROE: RAM.4, V10/4.Y
- removed net RWE: RAM.3, V10/3.Y
- removed net SL: ALU.5
- removed net SR: ALU.3
- removed net SUB: ALU.13, V37/2.Y
- removed net TCLR: TRING.1
- removed net XCP: REG.1, V1/1.Y
- removed net XOE: REG.3, V10/1.Y
- removed net XOR: ALU.7, V44/2.Y
- removed net YCP: REG.2, V1/2.Y
- removed net YOE: REG.4, V10/2.Y
- removed net ZF: FLAG.1, V55/2.A, V56/4.A
- new net CLR: PC-CLR.1, TRING.1
- net 0X00: now also V1/1.Y; no longer V28/1.Y
- net 0XFE: now also V4/2.Y; no longer V56/2.Y
- net 0XFF: now also V4/1.Y; no longer V56/1.Y
- net ADA: now also ALU-OP0.25; no longer V331.D, V351.C, V39/1.C, V491.D
- net ADI: now also ALU-OP0.24, PC-OP0.12, RAM-OP.5; no longer V141.D, V21/1.A, V28/3.B, V40/2.A, V46/3.B
- net ADV: now also ALU-OP0.23, PC-OP0.11; no longer V181.B, V30/1.A, V40/1.A, V47/3.A
- net ADX: now also ALU-OP0.27, REG-OP.22; no longer V331.B, V39/1.A, V491.A, V491.B, V61.C
- net ADY: now also ALU-OP0.26, REG-OP.21; no longer V331.C, V39/1.B, V491.C, V71.C
- net ANA: now also ALU-OP0.9; no longer V341.B, V351.G, V39/3.C
- net ANV: now also ALU-OP0.8, PC-OP0.2; no longer V181.G, V30/1.C, V40/5.A, V47/3.C
- net ANX: now also ALU-OP0.11, REG-OP.8; no longer V331.H, V39/3.A, V491.H, V61.G
- net ANY: now also ALU-OP0.10, REG-OP.7; no longer V341.A, V39/3.B, V71.G
- net CALL: now also PC-OP0.23, RAM-OP.16, V31.A; no longer V151.A, V531.A, V60/1.A, V60/1.B
- net CLA: now also ALU-OP0.30, V2/1.A; no longer V24/3.A, V29/2.A
- net CLK: now also ALU-CLK.1, PC-CLK.1, RAM-CLK.1, REG-CLK.1, V1/4.A; no longer V13/1.A, V13/2.A, V13/3.C, V17/1.C, V17/2.A, V2/1.A, V2/3.A, V24/1.B, V24/2.B, V29/1.B, V29/3.B, V3/1.A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
- net CLX: now also REG-OP.30, V2/1.B; no longer V2/2.A, V24/3.B
- net CLY: now also REG-OP.29, V2/1.C; no longer V24/3.C, V3/3.A
- net CMA: now also ALU-OP0.28; no longer V351.B, V50/3.C
- net CMV: now also PC-OP0.24; no longer V181.A
- net CMX: now also REG-OP.26; no longer V50/3.A, V61.B
- net CMY: now also REG-OP.25; no longer V50/3.B, V71.B
- net GND: now also ALU-PS.1, C4.-, C5.-, C6.-, C7.-, PC-PS.1, RAM-PS.1, REG-PS.1; no longer R2.1, V10/-UB.-UB, V11/-UB.-UB, V12/-UB.-UB, V13/-UB.-UB, V14/-UB.-UB, V15/-UB.-UB, V16/-UB.-UB, V17/-UB.-UB, V18/-UB.-UB, V19/-UB.-UB, V20/-UB.-UB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
- net HLT: now also CLK.1
- net IRCP: now also V1/4.Y; no longer V60/3.Y
- net JE: now also PC-OP0.14, RAM-OP.7, V31.G, V31.H; no longer V151.G, V151.H, V531.F, V55/6.A
- net JG: now also PC-OP0.16, RAM-OP.8, V31.E; no longer V151.F, V531.E, V55/5.A
- net JL: now also PC-OP0.15, RAM-OP.9, V31.F; no longer V151.E, V531.G, V531.H, V55/4.A
- net JN: now also PC-OP0.17, RAM-OP.10, V31.D; no longer V151.D, V531.D, V55/3.A
- net JNZ: now also PC-OP0.18, RAM-OP.11, V31.C; no longer V151.C, V531.C, V55/1.A
- net JZ: now also PC-OP0.19, RAM-OP.12, V31.B; no longer V151.B, V531.B, V54/4.A, V54/4.B
- net LDA: now also ALU-OP0.17, PC-OP0.6; no longer V181.F, V331.A
- net LDAI: now also ALU-OP0.16, PC-OP0.3, RAM-OP.1; no longer V141.H, V21/2.B, V21/2.C, V26/3.A
- net LDX: now also PC-OP0.8, REG-OP.18; no longer V181.D, V4/1.A
- net LDXI: now also PC-OP0.5, RAM-OP.3, REG-OP.16; no longer V141.F, V21/1.C, V4/2.A
- net LDY: now also PC-OP0.7, REG-OP.17; no longer V181.E, V4/3.A
- net LDYI: now also PC-OP0.4, RAM-OP.2, REG-OP.15; no longer V141.G, V21/2.A, V4/4.A
- net MAX: now also ALU-OP0.13, REG-OP.10; no longer V29/2.B, V61.F
- net MAY: now also ALU-OP0.12, REG-OP.9; no longer V29/2.C, V71.F
- net MXA: now also ALU-OP0.15, REG-OP.13; no longer V2/2.C, V351.E
- net MXY: now also REG-OP.14; no longer V2/2.B, V71.E
- net MYA: now also ALU-OP0.14, REG-OP.11; no longer V3/3.C, V351.F
- net MYX: now also REG-OP.12; no longer V3/3.B, V61.E
- net N$1: now also V1/1.B, V2/1.Y; no longer V10/2.A, V11/2.Y
- net N$10: now also V1/2.Y, V4/2.B; no longer V11/2.B, V9/2.Y
- net N$11: now also V2/2.Y, V4/1.B; no longer V8/2.Y, V9/2.B
- net N$12: now also V1/3.Y, V4/1.A; no longer V2/1.C, V2/2.Y
- net N$2: now also V2/2.C, V2/3.A, V31.Y; no longer V1/2.A, V3/2.Y
- net N$9: now also V2/3.Y, V4/2.A; no longer V2/3.C, V4/1.Y
- net NOA: now also ALU-OP1.2; no longer V27/2.B, V341.H, V42/2.C
- net NOV: now also ALU-OP1.1, PC-OP1.1; no longer V20/3.A, V30/2.B, V45/1.A, V48/1.B
- net NOX: now also ALU-OP1.4, REG-OP.2; no longer V341.F, V42/2.A, V8/1.A
- net NOY: now also ALU-OP1.3, REG-OP.1; no longer V341.G, V42/2.B, V8/2.A
- net ORA: now also ALU-OP0.5; no longer V341.E, V351.H, V42/1.C
- net ORV: now also ALU-OP0.4, PC-OP0.1; no longer V181.H, V30/2.A, V40/6.A, V48/1.A
- net ORX: now also ALU-OP0.7, REG-OP.6; no longer V341.C, V42/1.A, V61.H
- net ORY: now also ALU-OP0.6, REG-OP.5; no longer V341.D, V42/1.B, V71.H
- net OUA: now also ALU-OP0.29; no longer V351.A
- net OUX: now also REG-OP.28; no longer V61.A
- net OUY: now also REG-OP.27; no longer V71.A
- net RET: now also PC-OP0.13, RAM-OP.6, V1/2.A, V1/3.B; no longer V12/1.A, V12/2.A, V12/3.A, V26/1.A, V52/3.B, V52/3.C, V54/1.B, V54/2.B
- net STA: now also PC-OP0.20, RAM-OP.13; no longer V141.C, V17/3.C, V26/4.A
- net STX: now also PC-OP0.22, RAM-OP.15, REG-OP.24; no longer V141.A, V17/3.A, V4/5.A
- net STY: now also PC-OP0.21, RAM-OP.14, REG-OP.23; no longer V141.B, V17/3.B, V4/6.A
- net SUA: now also ALU-OP0.20; no longer V331.G, V351.D, V39/2.C, V491.G
- net SUI: now also ALU-OP0.19, PC-OP0.10, RAM-OP.4; no longer V141.E, V21/1.B, V28/3.A, V40/4.A, V46/3.A
- net SUV: now also ALU-OP0.18, PC-OP0.9; no longer V181.C, V30/1.B, V40/3.A, V47/3.B
- net SUX: now also ALU-OP0.22, REG-OP.20; no longer V331.E, V39/2.A, V491.E, V61.D
- net SUY: now also ALU-OP0.21, REG-OP.19; no longer V331.F, V39/2.B, V491.F, V71.D
- net T0: now also PC-T.10; no longer V62/1.B
- net T1: now also PC-T.9, V1/4.B; no longer V60/3.A, V63/1.A
- net T10: now also PC-T.1; no longer V54/3.A
- net T2: now also ALU-T.5, PC-T.8, RAM-T.8, REG-T.3, V1/1.A, V1/3.A; no longer V11/2.A, V16/2.A, V16/2.B, V17/2.B, V2/1.B, V27/3.B, V28/1.A, V29/1.A, V3/2.B, V38/1.A, V38/4.A, V41/4.A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
- net T3: now also ALU-T.4, PC-T.7, RAM-T.7, REG-T.2; no longer V13/1.B, V19/3.A, V2/3.B, V20/4.A, V24/1.A, V32/2.A, V38/2.A, V41/1.A, V41/3.A, V43/2.A, V43/4.A, V46/1.A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
- net T4: now also ALU-T.3, PC-T.6, RAM-T.6, V1/2.B; no longer V16/3.B, V16/3.C, V29/3.A, V46/4.B, V54/2.A, V9/3.A
- net T5: now also PC-T.5, RAM-T.5; no longer V17/1.B, V19/3.B, V21/3.B, V21/3.C, V24/2.A
- net T6: now also ALU-T.2, PC-T.4, RAM-T.4, REG-T.1, V2/2.A, V2/2.B; no longer V11/1.A, V11/3.B, V13/3.B, V20/2.A, V23/1.A, V28/4.A, V3/1.B, V30/3.A, V38/3.A, V41/2.A, V47/1.A, V5/2.B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
- net T7: now also ALU-T.1, PC-T.3, RAM-T.3; no longer V19/1.A, V23/3.B, V32/1.A, V51/1.A
- net T8: now also RAM-T.2, V2/3.B, V2/3.C; no longer V52/2.B, V52/2.C, V9/4.B
- net T9: now also PC-T.2, RAM-T.1; no longer V19/1.B, V23/4.B
- net VCC: now also ALU-PS.2, C4.+, C5.+, C6.+, C7.+, PC-PS.2, RAM-PS.2, REG-PS.2; no longer S1.S, S1.S1, V10/+UB.+UB, V11/+UB.+UB, V12/+UB.+UB, V13/+UB.+UB, V14/+UB.+UB, V15/+UB.+UB, V16/+UB.+UB, V17/+UB.+UB, V18/+UB.+UB, V19/+UB.+UB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
- net XOA: now also ALU-OP0.1; no longer V27/2.A, V32/3.C, V42/3.C
- net XOV: now also ALU-OP1.5, PC-OP1.2; no longer V20/3.B, V30/2.C, V45/2.A, V48/1.C
- net XOX: now also ALU-OP0.3, REG-OP.4; no longer V32/3.A, V42/3.A, V8/1.B
- net XOY: now also ALU-OP0.2, REG-OP.3; no longer V32/3.B, V42/3.B, V8/2.B

Commit message: LDO
Parts:
- added OCP: (no value), pinhead:PINHD-1X1
- added V5: 7410N, 74ttl-din:7410N
Connections:
- new net N$6: V5/1.C, V5/2.Y
- new net OCP: OCP.1, V5/1.Y
- net CLK: now also V5/1.B
- net GND: now also V5/-UB.-UB
- net OUA: now also V5/2.C
- net OUX: now also V5/2.A
- net OUY: now also V5/2.B
- net T2: now also V5/1.A
- net VCC: now also V5/+UB.+UB
Other:
- moved on the sheet: V1/4
Changed lines of the file:
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@@
 <drawing>
 <settings>
-<setting alwaysvectorfont="yes"/>
+<setting alwaysvectorfont="no"/>
 <setting verticaltext="up"/>
 </settings>
@@
 <part name="ALU-OP1" library="pinhead" library_urn="urn:adsk.eagle:library:325" deviceset="PINHD-1X5" device="" package3d_urn="urn:adsk.eagle:package:22469/2"/>
 <part name="ALU-OP0" library="pinhead" library_urn="urn:adsk.eagle:library:325" deviceset="PINHD-1X30" device="" package3d_urn="urn:adsk.eagle:package:22460/2"/>
+<part name="V5" library="74ttl-din" library_urn="urn:adsk.eagle:library:84" deviceset="74*10" device="N" package3d_urn="urn:adsk.eagle:package:16407/2"/>
+<part name="OCP" library="pinhead" library_urn="urn:adsk.eagle:library:325" deviceset="PINHD-1X1" device="" package3d_urn="urn:adsk.eagle:package:22485/2"/>
 </parts>
 <sheets>
@@
 <attribute name="VALUE" x="327.66" y="217.805" size="2.032" layer="96"/>
 </instance>
-<instance part="V1" gate="/4" x="304.8" y="109.22" smashed="yes">
-<attribute name="NAME" x="299.72" y="114.935" size="2.032" layer="95"/>
-<attribute name="VALUE" x="299.72" y="100.965" size="2.032" layer="96"/>
+<instance part="V1" gate="/4" x="256.54" y="165.1" smashed="yes">
+<attribute name="NAME" x="251.46" y="170.815" size="2.032" layer="95"/>
+<attribute name="VALUE" x="251.46" y="156.845" size="2.032" layer="96"/>
 </instance>
 <instance part="V2" gate="/1" x="322.58" y="243.84" smashed="yes">
@@
 <attribute name="NAME" x="161.29" y="108.585" size="1.778" layer="95" rot="R180"/>
 <attribute name="VALUE" x="161.29" y="190.5" size="1.778" layer="96" rot="R180"/>
+</instance>
+<instance part="V5" gate="/1" x="302.26" y="116.84" smashed="yes">
+<attribute name="NAME" x="297.18" y="125.095" size="2.032" layer="95"/>
+<attribute name="VALUE" x="297.18" y="106.045" size="2.032" layer="96"/>
+</instance>
+<instance part="V5" gate="/2" x="276.86" y="111.76" smashed="yes">
+<attribute name="NAME" x="271.78" y="120.015" size="2.032" layer="95"/>
+<attribute name="VALUE" x="271.78" y="100.965" size="2.032" layer="96"/>
+</instance>
+<instance part="V5" gate="/3" x="312.42" y="50.8" smashed="yes">
+<attribute name="NAME" x="307.34" y="59.055" size="2.032" layer="95"/>
+<attribute name="VALUE" x="307.34" y="40.005" size="2.032" layer="96"/>
+</instance>
+<instance part="OCP" gate="G$1" x="330.2" y="116.84" smashed="yes">
+<attribute name="NAME" x="323.85" y="120.015" size="1.778" layer="95"/>
+<attribute name="VALUE" x="323.85" y="111.76" size="1.778" layer="96"/>
+</instance>
+<instance part="V5" gate="/+UB" x="365.76" y="152.4" smashed="yes">
+<attribute name="NAME" x="367.03" y="151.13" size="1.524" layer="95"/>
+</instance>
+<instance part="V5" gate="/-UB" x="365.76" y="147.32" smashed="yes">
+<attribute name="NAME" x="367.03" y="147.32" size="1.524" layer="95"/>
 </instance>
 </instances>
@@
 <pinref part="ALU-T" gate="A" pin="5"/>
 <label x="162.56" y="210.82" size="1.778" layer="95" xref="yes"/>
+</segment>
+<segment>
+<pinref part="V5" gate="/1" pin="A"/>
+<wire x1="289.56" y1="121.92" x2="292.1" y2="121.92" width="0.1524" layer="91"/>
+<label x="289.56" y="121.92" size="1.778" layer="95" rot="R90" xref="yes"/>
 </segment>
 </net>
@@
 <wire x1="320.04" y1="154.94" x2="320.04" y2="157.48" width="0.1524" layer="91"/>
 <junction x="320.04" y="157.48"/>
+<pinref part="V5" gate="/+UB" pin="+UB"/>
+<wire x1="365.76" y1="154.94" x2="365.76" y2="157.48" width="0.1524" layer="91"/>
+<wire x1="365.76" y1="157.48" x2="363.22" y2="157.48" width="0.1524" layer="91"/>
 </segment>
 <segment>
@@
 <wire x1="320.04" y1="147.32" x2="320.04" y2="142.24" width="0.1524" layer="91"/>
 <junction x="320.04" y="142.24"/>
+<pinref part="V5" gate="/-UB" pin="-UB"/>
+<wire x1="365.76" y1="144.78" x2="365.76" y2="142.24" width="0.1524" layer="91"/>
+<wire x1="365.76" y1="142.24" x2="363.22" y2="142.24" width="0.1524" layer="91"/>
 </segment>
 <segment>
@@
 <segment>
 <pinref part="V1" gate="/4" pin="A"/>
-<wire x1="292.1" y1="111.76" x2="294.64" y2="111.76" width="0.1524" layer="91"/>
-<label x="292.1" y="111.76" size="1.778" layer="95" rot="R180" xref="yes"/>
+<wire x1="243.84" y1="167.64" x2="246.38" y2="167.64" width="0.1524" layer="91"/>
+<label x="243.84" y="167.64" size="1.778" layer="95" rot="R180" xref="yes"/>
+</segment>
+<segment>
+<pinref part="V5" gate="/1" pin="B"/>
+<wire x1="284.48" y1="116.84" x2="292.1" y2="116.84" width="0.1524" layer="91"/>
+<label x="284.48" y="116.84" size="1.778" layer="95" rot="R90" xref="yes"/>
 </segment>
 </net>
@@
 <label x="17.78" y="185.42" size="1.778" layer="95" xref="yes"/>
 </segment>
+<segment>
+<pinref part="V5" gate="/2" pin="A"/>
+<wire x1="264.16" y1="116.84" x2="266.7" y2="116.84" width="0.1524" layer="91"/>
+<label x="264.16" y="116.84" size="1.778" layer="95" rot="R180" xref="yes"/>
+</segment>
 </net>
 <net name="OUY" class="0">
@@
 <label x="33.02" y="182.88" size="1.778" layer="95" xref="yes"/>
 </segment>
+<segment>
+<pinref part="V5" gate="/2" pin="B"/>
+<wire x1="264.16" y1="111.76" x2="266.7" y2="111.76" width="0.1524" layer="91"/>
+<label x="264.16" y="111.76" size="1.778" layer="95" rot="R180" xref="yes"/>
+</segment>
 </net>
 <net name="CMY" class="0">
@@
 <segment>
 <pinref part="V1" gate="/4" pin="B"/>
-<wire x1="292.1" y1="106.68" x2="294.64" y2="106.68" width="0.1524" layer="91"/>
-<label x="292.1" y="106.68" size="1.778" layer="95" rot="R180" xref="yes"/>
+<wire x1="243.84" y1="162.56" x2="246.38" y2="162.56" width="0.1524" layer="91"/>
+<label x="243.84" y="162.56" size="1.778" layer="95" rot="R180" xref="yes"/>
 </segment>
 </net>
@@
 <label x="175.26" y="182.88" size="1.778" layer="95" xref="yes"/>
 </segment>
+<segment>
+<pinref part="V5" gate="/2" pin="C"/>
+<wire x1="264.16" y1="106.68" x2="266.7" y2="106.68" width="0.1524" layer="91"/>
+<label x="264.16" y="106.68" size="1.778" layer="95" rot="R180" xref="yes"/>
+</segment>
 </net>
 <net name="CMA" class="0">
@@
 <segment>
 <pinref part="V1" gate="/4" pin="Y"/>
-<wire x1="317.5" y1="109.22" x2="314.96" y2="109.22" width="0.1524" layer="91"/>
-<label x="317.5" y="109.22" size="1.778" layer="95" xref="yes"/>
-</segment>
-</net>
+<wire x1="269.24" y1="165.1" x2="266.7" y2="165.1" width="0.1524" layer="91"/>
+<label x="269.24" y="165.1" size="1.778" layer="95" xref="yes"/>
+</segment>
+</net>
+<net name="OCP" class="0">
+<segment>
+<pinref part="V5" gate="/1" pin="Y"/>
+<label x="314.96" y="116.84" size="1.778" layer="95" rot="R90" xref="yes"/>
+<pinref part="OCP" gate="G$1" pin="1"/>
+<wire x1="327.66" y1="116.84" x2="312.42" y2="116.84" width="0.1524" layer="91"/>
+</segment>
+</net>
+<net name="N$6" class="0">
+<segment>
+<pinref part="V5" gate="/2" pin="Y"/>
+<pinref part="V5" gate="/1" pin="C"/>
+<wire x1="287.02" y1="111.76" x2="292.1" y2="111.76" width="0.1524" layer="91"/>
+</segment>
+</net>
